Commit message: Fix mirrored thigh meshes for right legs

File: unitree_description/urdf/leg.xacro (robot description, xacro)
@@ -57,5 +57,5 @@
             <visual>
                 <geometry>
-                    <mesh filename="package://unitree_description/meshes/thigh.dae"
+                    <mesh filename="package://unitree_description/meshes/${'thigh.dae' if mirror == 1 else 'thigh_mirror.dae'}"
                           scale="1 1 1"/>
                 </geometry>
