Commit message: Add Go2 simulation, lidar and SLAM bridge setup

File: unitree_description/urdf/lidar.xacro (robot description, xacro)
@@ -20,5 +20,6 @@
     </joint>
     <gazebo reference="lidar_link">
-      <sensor name="lidar" type="lidar">
+      <sensor name="lidar" type="gpu_lidar">
+          <gz_frame_id>lidar_link</gz_frame_id>
         <pose relative_to="lidar_link">0 0 0 0 0 0</pose>
         <topic>/scan</topic>

File: unitree_description/urdf/unitree_go2_robot.xacro (robot description, xacro)
@@ -34,3 +34,24 @@
     <xacro:leg name="RR" mirror="-1" front_hind="-1"/>
     <xacro:lidar_sensor/>
+    <ros2_control name="Go2System" type="system">
+        <hardware><plugin>gz_ros2_control/GazeboSimSystem</plugin></hardware>
+        <joint name="FL_hip_joint"><command_interface name="position"/><state_interface name="position"/></joint>
+        <joint name="FL_upper_leg_joint"><command_interface name="position"/><state_interface name="position"/></joint>
+        <joint name="FL_lower_leg_joint"><command_interface name="position"/><state_interface name="position"/></joint>
+        <joint name="FR_hip_joint"><command_interface name="position"/><state_interface name="position"/></joint>
+        <joint name="FR_upper_leg_joint"><command_interface name="position"/><state_interface name="position"/></joint>
+        <joint name="FR_lower_leg_joint"><command_interface name="position"/><state_interface name="position"/></joint>
+        <joint name="RL_hip_joint"><command_interface name="position"/><state_interface name="position"/></joint>
+        <joint name="RL_upper_leg_joint"><command_interface name="position"/><state_interface name="position"/></joint>
+        <joint name="RL_lower_leg_joint"><command_interface name="position"/><state_interface name="position"/></joint>
+        <joint name="RR_hip_joint"><command_interface name="position"/><state_interface name="position"/></joint>
+        <joint name="RR_upper_leg_joint"><command_interface name="position"/><state_interface name="position"/></joint>
+        <joint name="RR_lower_leg_joint"><command_interface name="position"/><state_interface name="position"/></joint>
+    </ros2_control>
+    <gazebo>
+        <plugin filename="libgz_ros2_control-system.so"
+                name="gz_ros2_control::GazeboSimROS2ControlPlugin">
+            <parameters>$(find unitree_description)/config/controllers.yaml</parameters>
+        </plugin>
+    </gazebo>
 </robot>
